File: hardware/BLDC_Controller/BLDC_Controller.kicad_sch (KiCad schematic)
At the start: 61 parts, among them Q1 NMOS, Q2 NMOS, Q3 NMOS, Q4 NMOS, Q5 NMOS, Q6 NMOS, U1 STM32F405RGTx, U2 IR2103, U3 IR2103, U4 INA180A3, U5 INA180A3, U6 IR2103, U7 INA180A3

Commit message: Added potential 3.3V step down converter to schematic.
Parts:
- removed D7: D, symbol Device:D
- added C21, C24, C25: 22µ, symbol Device:C
- added C22: 1n, symbol Device:C
- added C23: 6.8n, symbol Device:C
- added C26, C34, C35: 2µ2, symbol Device:C
- added C27, C28, C29, C30, C31, C32, C33: 100n, symbol Device:C
- added C36, C37: 10p, symbol Device:C
- added IC1: MP2393GTL-Z, SOTFL50P160X60-8N, symbol MP2393GTL-Z:MP2393GTL-Z
- added L2: L, symbol Device:L
- added R21: 604k, symbol Device:R
- added R22: 20, symbol Device:R
- added R23: 25k, symbol Device:R
- added R24: 40.2k, symbol Device:R
- added R25: 13k, symbol Device:R
- added R26: R, symbol Device:R
- added Y2: 24MHz, symbol Device:Crystal_GND2
- C20: value C -> 1µ
- L1: value L -> 2.7µ
Connections:
- net BATT_SENSE is gone; now on net VCC_SENSE: C1.1, R1.2, R2.1
- net +3.3V: now also L1.2, U1.1 (VBAT), U1.19 (VDD), U1.32 (VDD), U1.48 (VDD), U1.64 (VDD), C24.2, C25.2, C26.2, C27.2, C28.2, C29.2, C30.2, C31.2, C32.2, L2.1, R24.2
- net CUR_SENSE_A: now also U1.20 (PA4)
- net CUR_SENSE_B: now also U1.22 (PA6)
- net CUR_SENSE_C: now also U1.24 (PC4)
- net GND: now also C1.2, R2.2, U1.12 (VSSA), U1.18 (VSS), U1.63 (VSS), C21.2, C22.2, C23.2, C24.1, C25.1, C26.1, C27.1, C28.1, C29.1, C30.1, C31.1, C32.1, C33.1, C34.1, C35.1, C36.1, C37.1, IC1.4 (GND), R25.1, Y2.2
- net HIN_A: now also U1.41 (PA8)
- net HIN_B: now also U1.42 (PA9)
- net HIN_C: now also U1.43 (PA10)
- net LIN_A: now also U1.23 (PA7)
- net LIN_B: now also U1.35 (PB14)
- net LIN_C: now also U1.36 (PB15)
- net VCC: now also C21.1, IC1.2 (IN), R21.1; no longer C20.1, L1.1
- net V_SENSE_A: now also U1.14 (PA0)
- net V_SENSE_B: now also U1.15 (PA1)
- net V_SENSE_C: now also U1.16 (PA2)
- net at U1.13 (VDDA): now also C33.2, L2.2
- net VCC_SENSE: now reaches U1.25 (PC5)
- net at U1.31 (VCAP_1): now also C34.2
- net at U1.47 (VCAP_2): now also C35.2
- net at U1.5 (PH0): now also C36.2, Y2.3
- net at U1.6 (PH1): now also R26.2
- new net: C22.1, IC1.1 (PG)
- new net: IC1.5 (BST), R22.1
- new net: C20.1, R22.2
- new net: IC1.6 (EN), R21.2
- new net: C20.2, IC1.3 (SW), L1.1
- new net: R23.2, R24.1, R25.2
- new net: C37.2, R26.1, Y2.1
- new net: C23.1, IC1.7 (SS)
- new net: IC1.8 (FB), R23.1
Other:
- note added: "FOC Electronic Speed Controller Design By: Kyle Tyni (github.com/kyletyni)"
- moved on the sheet: C1, R1, R2, U1
